File: date.kicad_sch (KiCad schematic)
At the start: 6 parts, among them U1 MAX7219

Commit message: Schéma/PCB : remplace le symbole des afficheurs CA56-12EWA par CC56-12EWA
Le schéma utilisait un symbole à anode commune alors que le câblage
(anodes communes CA1-CA4 vers les sorties DIG_x du MAX7219, qui
absorbent le courant) n'a de sens qu'avec des afficheurs à cathode
commune. Comme le circuit fonctionne, les composants montés sont bien
des CC56-12EWA.

Remplace le symbole dans date.kicad_sch et heure_alarme.kicad_sch (les
4 instances DATE1/ANNEE1/HEURE1/ALARME1), ainsi que la Value des
empreintes correspondantes dans reveil.kicad_pcb. Le footprint
(Display_7Segment:CA56-12EWA) et le datasheet sont inchangés : même
brochage, seules la doc et la BOM changent.

ERC/DRC revérifiés via le conteneur Docker KiBot : 0 erreur/avertissement
ERC, 6 avertissements DRC silk_edge_clearance sur J2 (inchangé,
préexistant), 0 écart schéma/PCB.

Co-Authored-By: Claude Sonnet 5 <noreply@anthropic.com>
Parts:
- ANNEE1, DATE1: value CA56-12EWA -> CC56-12EWA; symbol Display_Character:CA56-12EWA -> Display_Character:CC56-12EWA
Changed lines of the file:
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@@
 	)
 	(symbol
-		(lib_id "Display_Character:CA56-12EWA")
+		(lib_id "Display_Character:CC56-12EWA")
 		(at 152.4 88.9 0)
 		(unit 1)
@@
 			)
 		)
-		(property "Value" "CA56-12EWA"
+		(property "Value" "CC56-12EWA"
 			(at 152.4 73.66 0)
 			(effects
@@
 			)
 		)
-		(property "Description" "4 digit 7 segment high efficiency red LED, common anode"
+		(property "Description" "4 digit 7 segment high efficiency red LED, common cathode"
 			(at 152.4 88.9 0)
 			(effects
@@
 	)
 	(symbol
-		(lib_id "Display_Character:CA56-12EWA")
+		(lib_id "Display_Character:CC56-12EWA")
 		(at 228.6 88.9 0)
 		(unit 1)
@@
 			)
 		)
-		(property "Value" "CA56-12EWA"
+		(property "Value" "CC56-12EWA"
 			(at 228.6 73.66 0)
 			(effects
@@
 			)
 		)
-		(property "Description" "4 digit 7 segment high efficiency red LED, common anode"
+		(property "Description" "4 digit 7 segment high efficiency red LED, common cathode"
 			(at 228.6 88.9 0)
 			(effects

Commit message: Schéma/PCB : isole VBUS du jack J1, alimente le reste de la carte via VSYS
Le jack J1 alimentait directement le net VBUS, partagé avec la broche VBUS
du Pico : branché en même temps que l'USB, les deux 5 V se retrouvaient en
parallèle et le jack pouvait renvoyer du courant vers le PC.

Ajoute D3 (Schottky 1N5822, même référence que D2) entre le jack et un
nouveau rail renommé VSYS, plus C6 (220 µF) en entrée. Tout ce qui était
sur VBUS (MAX7219 U1/U2, moteur, LED, D2) passe sur VSYS, qui alimente le
Pico via sa broche VSYS (39) au lieu de VBUS (40) — VBUS reste réservé à
l'alimentation USB du Pico lui-même.

Met à jour le README (TODO alimentation + table des points de test).

Co-Authored-By: Claude Sonnet 5 <noreply@anthropic.com>
Connections:
- net VBUS renamed VSYS
Changed lines of the file:
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@@
 			)
 		)
-		(property "Value" "VBUS"
-			(at 83.82 154.94 0)
-			(effects
-				(font
-					(size 1.27 1.27)
-				)
+		(property "Value" "VSYS"
+			(at 86.36 158.7499 0)
+			(effects
+				(font
+					(size 1.27 1.27)
+				)
+				(justify left)
 			)
 		)
@@
 			)
 		)
-		(property "Value" "VBUS"
-			(at 71.12 62.23 0)
-			(effects
-				(font
-					(size 1.27 1.27)
-				)
+		(property "Value" "VSYS"
+			(at 73.66 66.0399 0)
+			(effects
+				(font
+					(size 1.27 1.27)
+				)
+				(justify left)
 			)
 		)
@@
 			)
 		)
-		(property "Value" "VBUS"
+		(property "Value" "VSYS"
 			(at 83.82 68.58 0)
 			(effects
